File: hw/sch_pcb/TFUNIPAYLOAD01.kicad_sch (KiCad schematic)
At the start: 71 parts, among them J1 SM08B-GHS-TB, J2 HEADER_2x15, J22 HEADER_2x03, J3 SM06B-GHS-TB, J7 SM03B-GHS-TB, M1 HOLE, M2 HOLE, M3 HOLE, M4 HOLE, Q2 BC817-25, Q3 BC817-25, Q4 BC817-25, U10 ATMEGA1284P-AU, U12 MIC5504-3.3YM5-TR, Y1 8 MHz

Commit message: Update schematics. Resolve #2
Parts:
- removed C26, C27, C28, C31, C36, C46, C51: 100nF, Capacitor_SMD:C_0805_2012Metric, symbol Device:C
- removed C41, C49: 10uF, Capacitor_SMD:C_0805_2012Metric, symbol Device:C
- removed D11: BZX585-B5V6.115, Diode_SMD:D_SOD-523, symbol MLAB_D:D_ZENER
- removed F2: SR010-15 100mA, Fuse:Fuse_0805_2012Metric, symbol Device:Polyfuse
- removed J22: HEADER_2x03, Mlab_Pin_Headers:SMD_2x03, symbol MLAB_HEADER:HEADER_2x03
- removed J7: SM03B-GHS-TB, Connector_JST:JST_GH_SM03B-GHS-TB_1x03-1MP_P1.25mm_Horizontal, symbol MLAB_CONNECTORS_JST:SM03B-GHS-TB
- removed JP4: Jumper_2_Bridged, NetTie:NetTie-2_SMD_Pad0.5mm, symbol Device:NetTie_2
- removed L1: NL03KT330, Inductor_SMD:L_0603_1608Metric_Pad1.05x0.95mm_HandSolder, symbol Device:L_Ferrite_Small
- removed TP5: Analog GND, TestPoint:TestPoint_Pad_D1.0mm, symbol Connector:TestPoint
- removed U12: MIC5504-3.3YM5-TR, Package_TO_SOT_SMD:SOT-23-5, symbol Regulator_Linear:MIC5504-3.3YM5
- added C13, C5: 22u, Capacitor_SMD:C_0805_2012Metric, symbol Device:C_Small
- added C14, C6: 47u, Capacitor_SMD:C_0805_2012Metric, symbol Device:C_Small
- added C15, C7: 10u, Capacitor_SMD:C_0805_2012Metric, symbol Device:C_Small
- added D7: RED, LED_SMD:LED_1206_3216Metric, symbol Device:LED
- added J3: HEADER_2x03, Mlab_Pin_Headers:SMD_2x03, symbol MLAB_HEADER:HEADER_2x03
- added J4: SM04B-GHS-TB, Connector_JST:JST_GH_SM04B-GHS-TB_1x04-1MP_P1.25mm_Horizontal, symbol MLAB_CONNECTORS_JST:SM04B-GHS-TB
- added J6: SM07B-GHS-TB, Connector_JST:JST_GH_SM07B-GHS-TB_1x07-1MP_P1.25mm_Horizontal, symbol ISM02A-rescue:SM07B-GHS-TB-MLAB_CONNECTORS_JST-ISM02A-rescue
- added L2, L3: 1uH - DFE252012P-1R0M=P2, Inductor_SMD:L_1008_2520Metric, symbol Device:L
- added R10: 511k, Resistor_SMD:R_0805_2012Metric, symbol Device:R_Small
- added R11, R23: 91k, Resistor_SMD:R_0805_2012Metric, symbol Device:R_Small
- added R2, R26, R3: 10k, Resistor_SMD:R_0805_2012Metric, symbol Device:R_Small
- added R22: 806k, Resistor_SMD:R_0805_2012Metric, symbol Device:R_Small
- added R24: 180R, Resistor_SMD:R_0805_2012Metric, symbol Device:R
- added R25, R27, R28, R29, R30: 100R, Resistor_SMD:R_0603_1608Metric, symbol Device:R
- added SW1: SKRTLAE010, Mlab_SW:SKRT, symbol MLAB_SW:SW_Push_shield
- added SW2, SW3: KMT031, Mlab_SW:KMT031 NGJ LHS C&K, symbol Switch:SW_Push
- added U1, U3: TPS631000DRLR, Package_TO_SOT_SMD:SOT-583-8, symbol MLAB_U:TPS631000DRLR
- renumbered C38 to C1, C34 to C10, C35 to C11, C39 to C12, C43 to C2, C30 to C3, C33 to C4, C40 to C8, C44 to C9, D6 to D1, D1 to D2, D9 to D3, D7 to D4, D10 to D5, D8 to D6, J3 to J1, J1 to J2, J2 to J5, L2 to L1, Q4 to Q1, R33 to R1, R20 to R12, R21 to R13, R38 to R14, R43 to R15, R37 to R16, R32 to R17, R41 to R18, R45 to R19, R46 to R20, R47 to R21, R34 to R4, R23 to R5, R44 to R6, R42 to R7, R36 to R8, R35 to R9, TP6 to TP1, TP7 to TP2, U10 to U2
Connections:
- net 3v3 is gone; now on net +3.3V: J5.5, J5.6
- net PB5 is gone; now on net MOSI: U2.1 ((PCINT13/MOSI)PB5)
- net PB6 is gone; now on net MISO: U2.2 ((PCINT14/MISO)PB6)
- net PB7 is gone; now on net SCLK: U2.3 ((PCINT15/SCK)PB7)
- net RST is gone; now on net ~{RST}_EXT: J5.10
- net connection_detector is gone; now on net EXT_DETECTION: J5.8
- net +3.3V: now also C6.1, C7.1, J3.2, R10.1, R2.1, R26.1, R3.1, U1.1 (VOUT)
- net GND: now also C8.2, C9.2, C13.2, C14.2, C15.2, C5.2, C6.2, C7.2, J3.6, J4.4, J4.MP, J6.7, J6.MP, R11.2, R23.2, R24.2, SW1.2, SW1.GND (SHIELD), SW2.2, SW3.1, U1.7 (GND), U3.7 (GND)
- net GNDA: no longer C8.2, C9.2
- net MISO: now also J3.1, R27.2
- net MOSI: now also J3.4, R28.2
- net SCL: now also J4.2
- net SCLK: now also J3.3
- net SDA: now also J4.3
- net BTN_USER_B: now reaches U2.30 ((PCINT7/ADC7)PA7)
- net BTN_USER_B: now also R3.2, SW2.1
- net BTN_USER_A: now reaches U2.31 ((PCINT6/ADC6)PA6)
- net BTN_USER_A: now also R2.2, SW1.1
- net #RTS: now reaches U2.32 ((PCINT5/ADC5)PA5)
- net #CTS: now reaches U2.33 ((PCINT4/ADC4)PA4)
- net EXT_DETECTION: now reaches U2.34 ((PCINT3/ADC3)PA3)
- net EXT_DETECTION: now also R26.2
- net EXT_B1: now reaches U2.41 ((PCINT9/CLKO/T1)PB1)
- net CS2: now reaches U2.43 ((PCINT11/AIN1/OC0)PB3)
- net CS2: now also R30.2
- net at C1.1, D2.1 (K), L1.1: now also D1.1 (K)
- net +VSW: now reaches L1.2
- net +VSW: now also C13.1, C5.1, U1.4 (VIN), U1.5 (EN), U1.6 (MODE), U3.4 (VIN), U3.5 (EN), U3.6 (MODE)
- net 5v renamed +5V
- net +5V: now also C14.1, C15.1, D7.2 (A), J4.1, J6.1, R22.1, U3.1 (VOUT)
- net External_5V: no longer names the net of D1.2 (A), J1.1
- net PB4 renamed CS1
- net CS1: now also R29.2
- net POWER_ANALOG_3V3: no longer names the net of U2.16 ((PCINT31/OC2A)PD7)
- net Signal: no longer names the net of U2.35 ((PCINT2/ADC2)PA2)
- net Signal_S&H renamed EXT_A0
- net Trace renamed EXT_B0
- net Virtual_ground renamed EXT_A1
- new net: D7.1 (K), R24.1
- new net: J6.2, R25.1
- new net: J6.3, R27.1
- new net: J6.4, R28.1
- new net: J6.5, R29.1
- new net: J6.6, R30.1
- new net: L2.2, U1.2 (LX2)
- new net: L2.1, U1.3 (LX1)
- new net: L3.2, U3.2 (LX2)
- new net: L3.1, U3.3 (LX1)
- new net 3v3i_FB: R10.2, R11.1, U1.8 (FB)
- new net 5v_FB: R22.2, R23.1, U3.8 (FB)
- new net RST#_P: J3.5, SW3.2
- new net SCK: R25.2
- no-connect marks 9 -> 4
Other:
- note added: "+3.3V"
- note added: "+5V"
- note added: "SPI - Dronecode Autopilot Connector Standard"
- note removed: "MISO"
- note removed: "MOSI"
- note removed: "SCK"
- note removed: "VTG"
- moved on the sheet: C1, C10, C11, C12, C8, C9, D1, D2, D4, D5, J1, J2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

Commit message: Fix ERC errors. Fix #3.
Parts:
- removed C3, C4: 15pF, Capacitor_SMD:C_0805_2012Metric, symbol Device:C
- removed Y1: 8 MHz, Mlab_XTAL:Crystal_HC49-4H_Vertical, symbol Device:Crystal
- added C3, C4: 15p, Capacitor_SMD:C_0805_2012Metric, symbol Device:C_Small
- added Y1: 8 MHz, Crystal:Crystal_SMD_3225-4Pin_3.2x2.5mm, symbol Device:Crystal_GND24_Small
- J6: symbol ISM02A-rescue:SM07B-GHS-TB-MLAB_CONNECTORS_JST-ISM02A-rescue -> MLAB_CONNECTORS_JST:SM07B-GHS-TB
- Q1, Q2, Q3: symbol Device:Q_NPN_BEC -> Transistor_BJT:BC817
- U2: symbol SPACEDOS01A_PCB01A-rescue:ATMEGA1284P-AU-atmel-DATALOGGER01A-rescue-CCP2019V01A-rescue -> MCU_Microchip_ATmega:ATmega1284P-A
Connections:
- net AVCC is gone; now on net +3.3V: U2.27 (AVCC)
- net EXT_A0 is gone; now on net A0: U2.37 (PA0)
- net EXT_A1 is gone; now on net A1: U2.36 (PA1)
- net EXT_B0 is gone; now on net B0: U2.40 (PB0)
- net EXT_B1 is gone; now on net B1: U2.41 (PB1)
- net GNDA is gone; now on net GND: U2.28 (GND)
- net I2C_PWR is gone; now on net +3.3V: J5.25, J5.26
- net RX is gone; now on net RX1: J5.12
- net SCK is gone; now on net SCLK: R25.2
- net TX is gone; now on net TX1: J5.14
- net #CTS: now also J1.5, JP1.2 (B)
- net #RTS: now also J1.4
- net C0: now also U2.21 (PC2)
- net C1: now also U2.16 (PD7)
- net GND: now also C3.2, C4.2, Y1.2, Y1.4
- net at U2.7 (XTAL2): now also C4.1, Y1.1
- net at U2.8 (XTAL1): now also C3.1, Y1.3
- no-connect marks 4 -> 2
Other:
- note added: "I²C - Dronecode Autopilot Connector Standard"
- note added: "ThunderFly TFGPS Payload Connector"
- moved on the sheet: C2, C8, C9, R12, R13, R5, TP1, TP2

Commit message: PCB layout WIP.
Parts:
- removed D1: BZX585-B5V6.115, Diode_SMD:D_SOD-523, symbol MLAB_D:D_ZENER
- removed SW1: SKRTLAE010, Mlab_SW:SKRT, symbol MLAB_SW:SW_Push_shield
- removed SW3: KMT031, Mlab_SW:KMT031 NGJ LHS C&K, symbol Switch:SW_Push
- added D1: BAS516, Diode_SMD:D_SOD-523, symbol Diode:BAS516
- added SW1: SKRTLAE010, Mlab_SW:KMT031 NGJ LHS C&K, symbol Switch:SW_Push
- D2: symbol MLAB_D:D_ZENER -> Device:D_Zener
- SW2: value KMT031 -> SKRTLAE010
Connections:
- net BTN_USER_A: now also SW1.1
- net GND: now also SW1.2
- net at J1.1: now also D1.2 (A)
- net at C1.1, D2.1 (K), L1.1: now also D1.1 (K)

Commit message: Components placement.
Parts:
- removed FID4, FID5, FID6: Fiducial, Fiducial:Fiducial_1mm_Mask2mm, symbol Mechanical:Fiducial
- J3: footprint Mlab_Pin_Headers:SMD_2x03 -> Mlab_Pin_Headers:SMD_2x03_WO_paste; now fitted

Commit message: Footprints updated.
Connections:
- net +5V: no longer J4.1, J6.1
- net +VSW: now also J4.1, J6.1
Other:
- note added: "Telemetry Peripheral Connector"
Changed lines of the file:
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@@
 		)
 	)
+	(text "Telemetry Peripheral\nConnector"
+		(exclude_from_sim no)
+		(at 25.654 22.352 0)
+		(effects
+			(font
+				(size 1.524 1.524)
+			)
+			(href "#1")
+		)
+	)
 	(text "+5V"
 		(exclude_from_sim no)
@@
 	(wire
 		(pts
+			(xy 265.43 176.53) (xy 265.43 180.34)
+		)
+		(stroke
+			(width 0)
+			(type solid)
+		)
+	)
+	(wire
+		(pts
 			(xy 29.21 160.02) (xy 44.45 160.02)
 		)
@@
 	)
 	(symbol
+		(lib_id "power:+VSW")
+		(at 265.43 176.53 0)
+		(unit 1)
+		(exclude_from_sim no)
+		(in_bom yes)
+		(on_board yes)
+		(dnp no)
+		(fields_autoplaced yes)
+		(property "Reference" "#PWR017"
+			(at 265.43 180.34 0)
+			(effects
+				(font
+					(size 1 1)
+				)
+				(hide yes)
+			)
+		)
+		(property "Value" "+VSW"
+			(at 265.43 172.72 0)
+			(effects
+				(font
+					(size 1 1)
+				)
+			)
+		)
+		(property "Footprint" ""
+			(at 265.43 176.53 0)
+			(effects
+				(font
+					(size 1 1)
+				)
+				(hide yes)
+			)
+		)
+		(property "Datasheet" ""
+			(at 265.43 176.53 0)
+			(effects
+				(font
+					(size 1 1)
+				)
+				(hide yes)
+			)
+		)
+		(property "Description" ""
+			(at 265.43 176.53 0)
+			(effects
+				(font
+					(size 1.27 1.27)
+				)
+				(hide yes)
+			)
+		)
+		(pin "1"
+		)
+		(instances
+			(project "TFUNIPAYLOAD01"
+				(path "/0a87ced0-2af2-43c5-a56c-218f7013d76f"
+					(reference "#PWR017")
+					(unit 1)
+				)
+			)
+		)
+	)
+	(symbol
 		(lib_id "power:GND")
 		(at 336.55 82.55 0)
@@
 	)
 	(symbol
-		(lib_id "power:+5V")
-		(at 265.43 213.36 0)
-		(mirror y)
-		(unit 1)
-		(exclude_from_sim no)
-		(in_bom yes)
-		(on_board yes)
-		(dnp no)
-		(property "Reference" "#PWR064"
-			(at 265.43 217.17 0)
-			(effects
-				(font
-					(size 1.27 1.27)
-				)
-				(hide yes)
-			)
-		)
-		(property "Value" "+5V"
-			(at 265.43 209.55 0)
-			(effects
-				(font
-					(size 1.27 1.27)
-				)
-			)
-		)
-		(property "Footprint" ""
-			(at 265.43 213.36 0)
-			(effects
-				(font
-					(size 1.27 1.27)
-				)
-				(hide yes)
-			)
-		)
-		(property "Datasheet" ""
-			(at 265.43 213.36 0)
-			(effects
-				(font
-					(size 1.27 1.27)
-				)
-				(hide yes)
-			)
-		)
-		(property "Description" ""
-			(at 265.43 213.36 0)
-			(effects
-				(font
-					(size 1.27 1.27)
-				)
-				(hide yes)
-			)
-		)
-		(pin "1"
-		)
-		(instances
-			(project "TFUNIPAYLOAD01"
-				(path "/0a87ced0-2af2-43c5-a56c-218f7013d76f"
-					(reference "#PWR064")
-					(unit 1)
-				)
-			)
-		)
-	)
-	(symbol
 		(lib_id "power:GND")
 		(at 270.51 41.91 0)
@@
 	)
 	(symbol
-		(lib_id "power:+5V")
-		(at 265.43 180.34 0)
+		(lib_id "power:GND")
+		(at 389.89 102.87 0)
 		(unit 1)
 		(exclude_from_sim no)
@@
 		(on_board yes)
 		(dnp no)
-		(property "Reference" "#PWR051"
-			(at 265.43 184.15 0)
+		(property "Reference" "#PWR022"
+			(at 389.89 109.22 0)
 			(effects
 				(font
@@
 			)
 		)
-		(property "Value" "+5V"
-			(at 265.811 175.9458 0)
+		(property "Value" "GND"
+			(at 390.0043 107.1944 0)
 			(effects
 				(font
@@
 		)
 		(property "Footprint" ""
-			(at 265.43 180.34 0)
+			(at 389.89 102.87 0)
 			(effects
 				(font
@@
 		)
 		(property "Datasheet" ""
-			(at 265.43 180.34 0)
+			(at 389.89 102.87 0)
 			(effects
 				(font
@@
 		)
 		(property "Description" ""
-			(at 265.43 180.34 0)
+			(at 389.89 102.87 0)
 			(effects
 				(font
@@
 			(project "TFUNIPAYLOAD01"
 				(path "/0a87ced0-2af2-43c5-a56c-218f7013d76f"
-					(reference "#PWR051")
+					(reference "#PWR022")
 					(unit 1)
 				)
@@
 	)
 	(symbol
-		(lib_id "power:GND")
-		(at 389.89 102.87 0)
+		(lib_id "power:+VSW")
+		(at 265.43 213.36 0)
 		(unit 1)
 		(exclude_from_sim no)
@@
 		(on_board yes)
 		(dnp no)
-		(property "Reference" "#PWR022"
-			(at 389.89 109.22 0)
+		(fields_autoplaced yes)
+		(property "Reference" "#PWR041"
+			(at 265.43 217.17 0)
 			(effects
 				(font
-					(size 1.27 1.27)
+					(size 1 1)
 				)
 				(hide yes)
 			)
 		)
-		(property "Value" "GND"
-			(at 390.0043 107.1944 0)
+		(property "Value" "+VSW"
+			(at 265.43 209.55 0)
 			(effects
 				(font
-					(size 1.27 1.27)
+					(size 1 1)
 				)
 			)
 		)
 		(property "Footprint" ""
-			(at 389.89 102.87 0)
+			(at 265.43 213.36 0)
 			(effects
 				(font
-					(size 1.27 1.27)
+					(size 1 1)
 				)
 				(hide yes)
@@
 		)
 		(property "Datasheet" ""
-			(at 389.89 102.87 0)
+			(at 265.43 213.36 0)
 			(effects
 				(font
-					(size 1.27 1.27)
+					(size 1 1)
 				)
 				(hide yes)
@@
 		)
 		(property "Description" ""
-			(at 389.89 102.87 0)
+			(at 265.43 213.36 0)
 			(effects
 				(font
@@
 			(project "TFUNIPAYLOAD01"
 				(path "/0a87ced0-2af2-43c5-a56c-218f7013d76f"
-					(reference "#PWR022")
+					(reference "#PWR041")
 					(unit 1)
 				)

Commit message: Routing.
Connections:
- net RST#_P is gone; now on net ~{RST}_PRG: J3.5
- net #CTS renamed ~{CTS}
- net #RTS renamed ~{RTS}
Changed lines of the file:
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@@
 		)
 	)
-	(label "#CTS"
+	(label "~{CTS}"
 		(at 36.83 39.37 180)
 		(effects
@@
 		)
 	)
+	(label "~{RST}_PRG"
+		(at 156.21 161.29 0)
+		(effects
+			(font
+				(size 1 1)
+			)
+			(justify left bottom)
+		)
+	)
 	(label "~{RST}_EXT"
 		(at 173.99 64.77 0)
@@
 		)
 	)
-	(label "RST#_P"
-		(at 156.21 161.29 0)
-		(effects
-			(font
-				(size 1 1)
-			)
-			(justify left bottom)
-		)
-	)
 	(label "TIMEPULSE"
 		(at 232.41 143.51 0)
@@
 		)
 	)
-	(label "#RTS"
+	(label "~{RTS}"
 		(at 240.03 77.47 180)
 		(effects
@@
 		)
 	)
-	(label "#RTS"
+	(label "~{RTS}"
 		(at 33.02 36.83 180)
 		(effects
@@
 		)
 	)
-	(label "#CTS"
+	(label "~{CTS}"
 		(at 240.03 74.93 180)
 		(effects

Commit message: Pinheader correctly positioned.
Parts:
- removed Q3: BC817-25, Package_TO_SOT_SMD:SOT-23, symbol Transistor_BJT:BC817
- removed R16: 10k, Resistor_SMD:R_0805_2012Metric, symbol Device:R
- D3, D4, D5, D6, D7: footprint LED_SMD:LED_1206_3216Metric -> Mlab_D:LED_1206_mill
- J5: footprint Connector_PinSocket_2.54mm:PinSocket_2x15_P2.54mm_Vertical -> Mlab_Pin_Headers:Straight_2x15
Connections:
- net Vin is gone; now on net +5V: D3.2 (A), D4.2 (A)
- net +3.3V: no longer D6.2 (A)
- net GND: now also D6.1 (K)
- net PC7_D3: now also R15.2
- net at R15.1: now also D6.2 (A)
Other:
- note added: "Transistors may be removed in future revision,"
- moved on the sheet: D6, R15
