File: hw/sch_pcb/TFUNIPAYLOAD01.kicad_pcb (KiCad board)
At the start: 2 copper layers, 70.6 x 50.3 mm, 80 parts, among them J1 SM06B-GHS-TB, J2 SM08B-GHS-TB, J3 HEADER_2x03, J4 SM04B-GHS-TB, J5 HEADER_2x15, J6 SM07B-GHS-TB, M1 HOLE, M2 HOLE, M3 HOLE, M4 HOLE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

Commit message: Adding Made in EU symbol.
Parts:
- added G***: LOGO, MLAB_LOGA:Made_in_EU, B.Cu at (159.8, 109.9)

Commit message: Fix LED resistors values.
Parts:
- R15: value 18R -> 100R
- R6: value 51R -> 100R
- R8: value 82R -> 180R
Changed lines of the file:
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@@
 			)
 		)
-		(property "Datasheet" "~"
+		(property "Datasheet" "https://v4.cecdn.yun300.cn/100001_2003185297/17%20FYLS-1206XXXC-D.pdf"
 			(at 0 0 0)
 			(layer "B.Fab")
@@
 			)
 		)
-		(property "Value" "51R"
+		(property "Value" "100R"
 			(at -0.4318 1.6256 0)
 			(layer "B.Fab")
@@
 			)
 		)
-		(property "UST_ID" "5c70984512875079b91f8953"
+		(property "UST_ID" "5c70984512875079b91f8956"
 			(at 267.111268 -34.573414 90)
 			(layer "B.Fab")
@@
 			)
 		)
-		(property "Value" "18R"
+		(property "Value" "100R"
 			(at 2.794 0.0254 0)
 			(layer "B.Fab")
@@
 			)
 		)
-		(property "UST_ID" "5c70984512875079b91f896e"
+		(property "UST_ID" "5c70984512875079b91f8956"
 			(at 272.191268 -39.653414 90)
 			(layer "B.Fab")
@@
 			)
 		)
-		(property "Value" "82R"
+		(property "Value" "180R"
 			(at -0.0508 1.5748 0)
 			(layer "B.Fab")
@@
 			)
 		)
-		(property "UST_ID" "5c70984512875079b91f8976"
+		(property "UST_ID" "5c70984512875079b91f897c"
 			(at 262.031268 -29.493414 90)
 			(layer "B.Fab")
@@
 			(keep_text_aligned yes)
 		)
-		(gr_text "70.612 mm"
+		(gr_text "2780 mils"
 			(at 148.5 71.846 0)
 			(layer "Cmts.User")
@@
 			(keep_text_aligned yes)
 		)
-		(gr_text "50.292 mm"
+		(gr_text "1980 mils"
 			(at 189.5648 104.999999 90)
 			(layer "Cmts.User")
@@
 			(keep_text_aligned yes)
 		)
-		(gr_text "40.64 mm"
+		(gr_text "1600 mils"
 			(at 108.996 105 90)
 			(layer "Cmts.User")
@@
 			(keep_text_aligned yes)
 		)
-		(gr_text "60.96 mm"
+		(gr_text "2400 mils"
 			(at 148.5 132.4504 0)
 			(layer "Cmts.User")
